Commit message: Update frame references to lrmate_200id_world in camera_bridge_node, fanuc_bridge_node, follow_path_action, move_to_server, and URDF description

File: lrmate_200id_model_description/lrmate_200id/urdf/lrmate_200id_description.urdf.xacro (robot description, xacro)
@@ -103,4 +103,5 @@
       izz="3.1628E-05"
   />
+  <link name="lrmate_200id_world"/>
   <link name="ft_frame"/>
   <link name="tool0"/>
@@ -111,4 +112,10 @@
     <origin xyz="0 0 0" rpy="0 0 0"/>
     <axis xyz="0 0 1"/>
+  </joint>
+  <!-- This joint is used to transform from the world frame to the robot's base frame -->
+  <joint name="base_to_fanuc_world" type="fixed">
+    <parent link="base_link"/>
+    <child link="lrmate_200id_world"/>
+    <origin xyz="0 0 0.169" rpy="0 0 0"/>
   </joint>
   <!-- joints - main serial chain -->

Commit message: Adjust URDF according to the Standard DH table

File: lrmate_200id_model_description/lrmate_200id/urdf/lrmate_200id_description.urdf.xacro (robot description, xacro)
@@ -20,5 +20,5 @@
   <xacro:create_link
       link_name="link_1"
-      xyz_offset="0 0 0"
+      xyz_offset="0 0 -0.126259"
       rpy_offset="0 0 0"
       mesh_package="lrmate_200id_model_description/lrmate_200id"
@@ -62,5 +62,5 @@
   <xacro:create_link
       link_name="link_4"
-      xyz_offset="0 0 0"
+      xyz_offset="0.088001 0 0.035027"
       rpy_offset="0 0 0"
       mesh_package="lrmate_200id_model_description/lrmate_200id"
@@ -76,5 +76,5 @@
   <xacro:create_link
       link_name="link_5"
-      xyz_offset="0 0 0"
+      xyz_offset="-0.001599 0 0.035027"
       rpy_offset="0 0 0"
       mesh_package="lrmate_200id_model_description/lrmate_200id"
@@ -90,5 +90,5 @@
   <xacro:create_link
       link_name="link_6"
-      xyz_offset="0 0 0"
+      xyz_offset="0.048401 0 0.035027"
       rpy_offset="0 0 0"
       mesh_package="lrmate_200id_model_description/lrmate_200id"
@@ -117,20 +117,20 @@
     <parent link="base_link"/>
     <child link="lrmate_200id_world"/>
-    <origin xyz="0 0 0.169" rpy="0 0 0"/>
+    <origin xyz="0 0 0.33" rpy="0 0 0"/>
   </joint>
   <!-- joints - main serial chain -->
-  <joint name="joint_1" type="revolute">
+  <joint name="joint_1" type="revolute">k
     <parent link="base_link"/>
     <child link="link_1"/>
-    <origin xyz="0 0 0.042741" rpy="0 0 0"/>
+    <origin xyz="0 0 0.169" rpy="0 0 0"/>
     <axis xyz="0 0 1"/>
     <!-- according to official specs ${340.0 / 2.0 * pi / 180.0}-->
-    <limit effort="16.6" lower="-2.9671" upper="2.9671" velocity="5.93"/>
+    <limit effort="16.6" lower="${radians(-170)}" upper="2.9671" velocity="5.93"/>
   </joint>
   <joint name="joint_2" type="revolute">
     <parent link="link_1"/>
     <child link="link_2"/>
-    <origin xyz="0.05 0 0.28726" rpy="0 0 0"/>
-    <axis xyz="0 1 0"/>
+    <origin xyz="0.05 0 0.161" rpy="0 0 0"/>
+    <axis xyz="0 -1 0"/>
     <limit effort="16.6" lower="-1.7453" upper="2.5307" velocity="4.28"/>
   </joint>
@@ -145,5 +145,5 @@
     <parent link="link_3"/>
     <child link="link_4"/>
-    <origin xyz="0.088001 0 0.035027" rpy="0 0 0"/>
+    <origin xyz="0 0 0" rpy="0 0 0"/>
     <axis xyz="-1 0 0"/>
     <limit effort="16.6" lower="-3.3161" upper="3.3161" velocity="6.63"/>
@@ -152,5 +152,5 @@
     <parent link="link_4"/>
     <child link="link_5"/>
-    <origin xyz="0.2454 0 0" rpy="0 0 0"/>
+    <origin xyz="0.335 0 0" rpy="0 0 0"/>
     <axis xyz="0 -1 0"/>
     <limit effort="16.6" lower="-2.1817" upper="2.1817" velocity="4.36"/>
@@ -159,5 +159,5 @@
     <parent link="link_5"/>
     <child link="link_6"/>
-    <origin xyz="0.05 0 0" rpy="1.5708 0 0"/>
+    <origin xyz="0 0 0" rpy="1.5708 0 0"/>
     <axis xyz="-1 0 0"/>
     <limit effort="9.4" lower="-6.2832" upper="6.2832" velocity="12.57"/>

Commit message: modify lrmate_200id_model_description Referenced two files - One is a URDF generated using SolidWorks - The other is fanuc_lrmate200id_support/urdf/lrmate200id_macro.xacro The joints are written according to fanuc_lrmate200id_support, and the mesh offsets are balanced using SolidWorks

File: lrmate_200id_model_description/lrmate_200id/urdf/lrmate_200id_description.urdf.xacro (robot description, xacro)
@@ -20,5 +20,5 @@
   <xacro:create_link
       link_name="link_1"
-      xyz_offset="0 0 -0.126259"
+      xyz_offset="0 0 -0.287259"
       rpy_offset="0 0 0"
       mesh_package="lrmate_200id_model_description/lrmate_200id"
@@ -62,5 +62,5 @@
   <xacro:create_link
       link_name="link_4"
-      xyz_offset="0.088001 0 0.035027"
+      xyz_offset="0.088001 0 0"
       rpy_offset="0 0 0"
       mesh_package="lrmate_200id_model_description/lrmate_200id"
@@ -76,5 +76,5 @@
   <xacro:create_link
       link_name="link_5"
-      xyz_offset="-0.001599 0 0.035027"
+      xyz_offset="0 0 0"
       rpy_offset="0 0 0"
       mesh_package="lrmate_200id_model_description/lrmate_200id"
@@ -90,5 +90,5 @@
   <xacro:create_link
       link_name="link_6"
-      xyz_offset="0.048401 0 0.035027"
+      xyz_offset="-0.03 0 0"
       rpy_offset="0 0 0"
       mesh_package="lrmate_200id_model_description/lrmate_200id"
@@ -103,7 +103,4 @@
       izz="3.1628E-05"
   />
-  <link name="lrmate_200id_world"/>
-  <link name="ft_frame"/>
-  <link name="tool0"/>
   <!-- base_joint fixes base_link to the environment -->
   <joint name="base_joint" type="fixed">
@@ -114,4 +111,5 @@
   </joint>
   <!-- This joint is used to transform from the world frame to the robot's base frame -->
+  <link name="lrmate_200id_world"/>
   <joint name="base_to_fanuc_world" type="fixed">
     <parent link="base_link"/>
@@ -123,5 +121,5 @@
     <parent link="base_link"/>
     <child link="link_1"/>
-    <origin xyz="0 0 0.169" rpy="0 0 0"/>
+    <origin xyz="0 0 0.33" rpy="0 0 0"/>
     <axis xyz="0 0 1"/>
     <!-- according to official specs ${340.0 / 2.0 * pi / 180.0}-->
@@ -131,6 +129,6 @@
     <parent link="link_1"/>
     <child link="link_2"/>
-    <origin xyz="0.05 0 0.161" rpy="0 0 0"/>
-    <axis xyz="0 -1 0"/>
+    <origin xyz="0.050 0 0" rpy="0 0 0"/>
+    <axis xyz="0 1 0"/>
     <limit effort="16.6" lower="-1.7453" upper="2.5307" velocity="4.28"/>
   </joint>
@@ -145,5 +143,5 @@
     <parent link="link_3"/>
     <child link="link_4"/>
-    <origin xyz="0 0 0" rpy="0 0 0"/>
+    <origin xyz="0 0 0.035027" rpy="0 0 0"/>
     <axis xyz="-1 0 0"/>
     <limit effort="16.6" lower="-3.3161" upper="3.3161" velocity="6.63"/>
@@ -159,17 +157,21 @@
     <parent link="link_5"/>
     <child link="link_6"/>
-    <origin xyz="0 0 0" rpy="1.5708 0 0"/>
+    <origin xyz="0.080 0 0" rpy="0 0 0"/>
     <axis xyz="-1 0 0"/>
     <limit effort="9.4" lower="-6.2832" upper="6.2832" velocity="12.57"/>
   </joint>
-  <joint name="joint-ft_frame" type="fixed">
+  <!-- ROS-Industrial 'flange' frame: attachment point for EEF models -->
+  <link name="flange"/>
+  <joint name="link_6-flange" type="fixed">
     <parent link="link_6"/>
-    <child link="ft_frame"/>
+    <child link="flange"/>
     <origin xyz="0 0 0" rpy="0 0 0"/>
   </joint>
-  <joint name="joint-tool" type="fixed">
-    <parent link="ft_frame"/>
+  <!-- ROS-Industrial 'tool0' frame: all-zeros tool frame -->
+  <link name="tool0"/>
+  <joint name="flange-tool0" type="fixed">
+    <parent link="flange"/>
     <child link="tool0"/>
-    <origin xyz="0 0 .185" rpy="0 0 0"/>
+    <origin xyz="0 0 0" rpy="${pi} ${-pi/2.0} 0"/>
   </joint>
 </xacro:macro>

Commit message: add lrmate_200id_moveit_config(msa generated) replace lrmate_200id lrmate_200id_moveit_config can loaded by pilz(follow_path request)

File: lrmate_200id_model_description/lrmate_200id/urdf/lrmate_200id_description.urdf.xacro (robot description, xacro)
@@ -118,5 +118,5 @@
   </joint>
   <!-- joints - main serial chain -->
-  <joint name="joint_1" type="revolute">k
+  <joint name="joint_1" type="revolute">
     <parent link="base_link"/>
     <child link="link_1"/>
